File: KiCAD/KiCAD.kicad_pcb (KiCad board)
At the start: 2 copper layers, 50 x 50 mm, 12 parts, among them J1 RC Channel: Throttle, J2 RC Channel: Steering, J3 RC Channel: Emergency Stop, M1 Motor Controller, M2 Linear Actuator/Servo

Commit message: update photos and readme
Connections:
- net /5V renamed 5V
- net /GND renamed GND
- net Net-(A1-A0) renamed Steering Center Adjustment
- net Net-(A1-A1) renamed Steering Range Adjustment
- net Net-(A1-A2) renamed Speed Control
- net Net-(A1-A6) renamed Joystick Steering
- net Net-(A1-D3) renamed Motor Control
- net Net-(A1-D5) renamed Steering Control
- net Net-(A1-D7) renamed RC E-Stop
- net Net-(A1-D8) renamed RC Steering
- net Net-(A1-D9) renamed RC Throttle
- net Net-(A1-SDA/A4) renamed Joystick Throttle
- net Net-(A1-VIN) renamed Arduino Power Input
